File: miniSpartan6+_Rev_B.sch (EAGLE design)
At the start: 101 parts, among them J2 HDMI-TYPE-A-RECEPTICALFCI1002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, J3 HDMI-TYPE-A-RECEPTICALFCI1002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, J4 P24-1, J5 MICROSD_MOLEX, J6 P24-1, Q1 12MHz, U1 93C46B, U10 SPI_FLASH-SOIC_150_208, U11 PCA9306, U2 FT2232HL, U3 ADC088S102CIMT, U4 +3.3V Reg., U5 +1.2V Reg., U6 XC6SLX25-FT256, U7 ASFLMB-32.000MHZ-LC-T, U8 ASFLMB-50.000MHZ-LC-T, U9 SDRAM-16MX16-WINBOND, X1 MINI-USB-UX60-MB-5S8

Commit message: Revert "Merge remote-tracking branch 'scarabhardware/master'"
This reverts commit b5789720bcce7dd5b7e874fc360775f4b6e4c3f3, reversing
changes made to 397d36b8f68ee444c3233c14a563200e9bae67a6.
Other:
- note removed: "Copyright Scarab Hardware 2014 With some parts from Saanlima Electronics Under Creative Commons Attribution Sharealike 4.0"
- moved on the sheet: C16, C17, C18, C19, C20, C21, C22, C23, C24, C25, C26, C27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
